File: SynCrystal-kicad/ESS_in.kicad_sch (KiCad schematic)
At the start: 17 parts, among them Q2 SS8050, U1 74HCT14, U8 LMC6482

Commit message: Projector PCB!
Changed lines of the file:
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@@
-		)
-	)
-	(label "INT1"
-		(at 173.99 91.44 270)
-		(effects
-			(font
-				(size 1.27 1.27)
-			)
-			(justify right bottom)
 		)
 	)
@@
 		(effects
 			(font
+				(size 1.27 1.27)
+			)
+			(justify right)
+		)
+	)
+	(hierarchical_label "INT1"
+		(shape output)
+		(at 173.99 91.44 270)
+		(effects
+			(font
