File: SynCrystal-kicad/SynCrystal-kicad.kicad_sch (KiCad schematic)
At the start: 20 parts, among them CN1 PJ-342, J1 ICSP, J2 DIN-6 Male, SW5 Shaft_Pulses, U2 ATmega328P-A

Commit message: More changes
Parts:
- removed TP13: D, TestPoint:TestPoint_Pad_D1.0mm, symbol Peacemans Teile:TestPoint_named
- added D3: OLED 128x64, Peacemans Teile:OLED_128x63_i2c_0.96, symbol Peacemans Teile:OLED-128-64-I2C-Display_Character
- added JP1: VCC Ctrl, Jumper:SolderJumper-3_P1.3mm_Bridged2Bar12_RoundedPad1.0x1.5mm, symbol Jumper:SolderJumper_3_Bridged12
- added JP2: GND Ctrl, Jumper:SolderJumper-3_P1.3mm_Bridged2Bar12_RoundedPad1.0x1.5mm, symbol Jumper:SolderJumper_3_Bridged12
- added SW1: Mode -, Button_Switch_SMD:SW_SPST_PTS647_Sx50, symbol Switch:SW_Push
- added SW2: Mode +, Button_Switch_SMD:SW_SPST_PTS647_Sx50, symbol Switch:SW_Push
- added SW3: Frame -, Button_Switch_SMD:SW_SPST_PTS647_Sx50, symbol Switch:SW_Push
- added SW4: Frame +, Button_Switch_SMD:SW_SPST_PTS647_Sx50, symbol Switch:SW_Push
- SW5: value Shaft_Pulses -> Shaft_Pulse_Ratio
Connections:
- net +5V: now also JP1.2 (C)
- net Frame+: now also SW4.2
- net Frame-: now also SW3.2
- net GND: now also JP1.3 (B), JP2.2 (C), SW1.1, SW2.1, SW3.1, SW4.1
- net MISO: no longer TP6.1
- net MOSI: now also TP6.1
- net Mode+: now also SW2.2
- net Mode-: now also SW1.2
- net SCL: now also D3.3 (SCL)
- net SDA: now also D3.4 (SDA)
- net Proj_starting renamed IRSEND
- new net: D3.1 (GND), JP2.1 (A)
- new net: D3.2 (VCC), JP1.1 (A), JP2.3 (B)
Other:
- added sheet GuideStart (GuideStart.kicad_sch)
- sheet Frontpanel UI ports: added none; removed Frame+, Frame-, Mode+, Mode-
- note added: "To Do: - Frontpanel separieren - Guide/Follow Selector - INT1 wegsparen? (2 Schottkys) - Startpiepser statt ESS Impulen erkennen"
- note removed: "To Do: - Lampenrelais-Platine separieren - Frontpanel separieren - IR Receive - IR Out - Guide/Follow Selector - INT1 wegsparen? (2 Schottkys) - Startpiepser statt ESS Impulen erkennen"
- moved on the sheet: C1, J1, J3, R1, R12, R2, R25, R26, R3, SW5, U2
