File: SynCrystal-kicad/DAC.kicad_sch (KiCad schematic)
At the start: 11 parts, among them U6 MCP4725, U8 LMC6482

Commit message: Projector PCB!
Parts:
- added unit 3 of U8
Connections:
- net +5V: now also U8.8 (V+)
- net GND: now also U8.4 (V-)
Changed lines of the file:
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@@
+	)
+	(symbol
+		(lib_id "Amplifier_Operational:LMC6482")
+		(at 144.78 130.81 90)
+		(unit 3)
+		(exclude_from_sim no)
+		(in_bom yes)
+		(on_board yes)
+		(dnp no)
+		(property "Reference" "U8"
+			(at 143.764 135.89 90)
+			(effects
+				(font
+					(size 1.27 1.27)
+				)
+			)
+		)
+		(property "Value" "LMC6482"
+			(at 143.764 138.43 90)
+			(effects
+				(font
+					(size 1.27 1.27)
+				)
+			)
+		)
+		(property "Footprint" "Package_SO:SOIC-8_3.9x4.9mm_P1.27mm"
+			(at 144.78 130.81 0)
+			(effects
+				(font
+					(size 1.27 1.27)
+				)
+				(hide yes)
+			)
+		)
+		(property "Datasheet" "http://www.ti.com/lit/ds/symlink/lmc6482.pdf"
+			(at 144.78 130.81 0)
+			(effects
+				(font
+					(size 1.27 1.27)
+				)
+				(hide yes)
+			)
+		)
+		(property "Description" "Dual CMOS Rail-to-Rail Input and Output Operational Amplifier, DIP-8/SOIC-8, SSOP-8"
+			(at 144.78 130.81 0)
+			(effects
+				(font
+					(size 1.27 1.27)
+				)
+				(hide yes)
+			)
+		)
+		(pin "2"
+		)
+		(pin "7"
+		)
+		(pin "3"
+		)
+		(pin "4"
+		)
+		(pin "5"
+		)
+		(pin "8"
+		)
+		(pin "1"
+		)
+		(pin "6"
+		)
+		(instances
+			(project "SynCrystal-kicad"
+				(path "/904e3c46-2ed3-4778-9ca9-733b218304b0/c7c1d309-2c22-437c-b7c3-6ae7e0806726"
+					(reference "U8")
+					(unit 3)
+				)
+			)
+		)
 	)
 	(symbol
@@
 	(symbol
 		(lib_id "power:GNDD")
+		(at 152.4 133.35 0)
+		(unit 1)
+		(exclude_from_sim no)
+		(in_bom yes)
+		(on_board yes)
+		(dnp no)
+		(property "Reference" "#PWR032"
+			(at 152.4 139.7 0)
+			(effects
+				(font
+					(size 1.27 1.27)
+				)
+				(hide yes)
+			)
+		)
+		(property "Value" "GND"
+			(at 152.4 137.16 0)
+			(effects
+				(font
+					(size 1.27 1.27)
+				)
+			)
+		)
+		(property "Footprint" ""
+			(at 152.4 133.35 0)
+			(effects
+				(font
+					(size 1.27 1.27)
+				)
+				(hide yes)
+			)
+		)
+		(property "Datasheet" ""
+			(at 152.4 133.35 0)
+			(effects
+				(font
+					(size 1.27 1.27)
+				)
+				(hide yes)
+			)
+		)
+		(property "Description" "Power symbol creates a global label with name \"GNDD\" , digital ground"
+			(at 152.4 133.35 0)
+			(effects
+				(font
+					(size 1.27 1.27)
+				)
+				(hide yes)
+			)
+		)
+		(pin "1"
+		)
+		(instances
+			(project "SynCrystal-kicad"
+				(path "/904e3c46-2ed3-4778-9ca9-733b218304b0/c7c1d309-2c22-437c-b7c3-6ae7e0806726"
+					(reference "#PWR032")
+					(unit 1)
+				)
+			)
+		)
+	)
+	(symbol
+		(lib_id "power:GNDD")
 		(at 127 102.87 0)
 		(unit 1)
@@
 					(unit 1)
 				)
+			)
+		)
+	)
+	(symbol
+		(lib_id "power:+5V")
+		(at 137.16 133.35 0)
+		(unit 1)
+		(exclude_from_sim no)
+		(in_bom yes)
+		(on_board yes)
+		(dnp no)
+		(property "Reference" "#PWR029"
+			(at 137.16 137.16 0)
+			(effects
+				(font
+					(size 1.27 1.27)
+				)
+				(hide yes)
+			)
+		)
+		(property "Value" "+5V"
+			(at 136.398 129.032 0)
+			(effects
+				(font
+					(size 1.27 1.27)
+				)
+			)
+		)
+		(property "Footprint" ""
+			(at 137.16 133.35 0)
+			(effects
+				(font
+					(size 1.27 1.27)
+				)
+				(hide yes)
+			)
+		)
+		(property "Datasheet" ""
+			(at 137.16 133.35 0)
+			(effects
+				(font
+					(size 1.27 1.27)
+				)
+				(hide yes)
+			)
+		)
+		(property "Description" "Power symbol creates a global label with name \"+5V\""
+			(at 137.16 133.35 0)
+			(effects
+				(font
+					(size 1.27 1.27)
+				)
+				(hide yes)
+			)
+		)
+		(pin "1"
+		)
+		(instances
+			(project "SynCrystal-kicad"
+				(path "/904e3c46-2ed3-4778-9ca9-733b218304b0/c7c1d309-2c22-437c-b7c3-6ae7e0806726"
+					(reference "#PWR029")
+					(unit 1)
+				)

Commit message: Starting to assign part numbers
Parts:
- removed C10: 1u, Capacitor_SMD:C_0603_1608Metric, symbol Device:C_Small
- removed C11: 100n, Capacitor_SMD:C_0603_1608Metric, symbol Device:C_Small
- removed R10: 4k7, Resistor_SMD:R_0603_1608Metric, symbol Device:R_Small
- removed R14: 2k7, Resistor_SMD:R_0603_1608Metric, symbol Device:R_Small
- removed R6, R9: 10k, Resistor_SMD:R_0603_1608Metric, symbol Device:R_Small
- removed RV2: 300, easyEDA:RES-SMD_RK10J11R0A0H, symbol Device:R_Potentiometer_Small
- removed TP12: 678, TestPoint:TestPoint_Pad_D1.0mm, symbol Peacemans Teile:TestPoint_named
- removed TP9: DAC, TestPoint:TestPoint_Pad_D1.0mm, symbol Peacemans Teile:TestPoint_named
- removed U6: MCP4725, Package_TO_SOT_SMD:SOT-23-6, symbol Analog_DAC:MCP4725xxx-xCH
- removed U8: LMC6482, Package_SO:SOIC-8_3.9x4.9mm_P1.27mm, symbol Amplifier_Operational:LMC6482
Connections:
- no-connect marks 1 -> 0
Other:
- note removed: "0.55-1.95V"
- note removed: "Für 0,5-1,5V: R9 12k, R14 2k2 Für 0.6-1.9V: R9 10k, R14 2k8"
