File: SynCrystal-kicad/Proj_Imp_Cleanup.kicad_sch (KiCad schematic)
At the start: 8 parts, among them Q1 SS8050, U1 74HCT14

Commit message: Projector PCB!
Parts:
- added C8: 100n, Capacitor_SMD:C_0603_1608Metric, symbol Device:C_Small
- added unit 7 of U1
Connections:
- net +5V: now also C8.2, U1.14 (VCC)
- net GND: now also C8.1, U1.7 (GND)

Commit message: Starting to assign part numbers
Parts:
- removed C12, C8: 100n, Capacitor_SMD:C_0603_1608Metric, symbol Device:C_Small
- removed Q1: SS8050, Package_TO_SOT_SMD:SOT-23, symbol Transistor_BJT:BC847
- removed R11, R15: 3k3, Resistor_SMD:R_0603_1608Metric, symbol Device:R_Small
- removed R5: 10k, Resistor_SMD:R_0603_1608Metric, symbol Device:R_Small
- removed R7: 47k, Resistor_SMD:R_0603_1608Metric, symbol Device:R_Small
- removed R8: 470k, Resistor_SMD:R_0603_1608Metric, symbol Device:R_Small
- removed U1: 74HCT14, Package_SO:TSSOP-14_4.4x5mm_P0.65mm, symbol Peacemans Teile:74HCT14
