File: SynCrystal-kicad/tcxo.kicad_sch (KiCad schematic)
At the start: 3 parts, among them U1 74HCT14, U4 ECS-TXO-3225MV-160-TR

Commit message: Starting to assign part numbers
Parts:
- removed C4: 100n, Capacitor_SMD:C_0603_1608Metric, symbol Device:C_Small
- removed U1: 74HCT14, Package_SO:TSSOP-14_4.4x5mm_P0.65mm, symbol Peacemans Teile:74HCT14
- removed U4: ECS-TXO-3225MV-160-TR, Crystal:Crystal_SMD_3225-4Pin_3.2x2.5mm, symbol easyEDA:ECS-TXO-3225MV-160-TR
