File: SynCrystal_ProjectorBoard/Projector_PCB.kicad_sch (KiCad schematic)
At the start: 20 parts, among them J10 Screw_Terminal_01x03, J11 to DIN Traces, J5 Relais Board, J6 uC Cable, J7 to DIN Connector, J8 to Motor Ctrl PCB, J9 to Motor Controller Hat, SW6 SW_SPDT, U10 AP63205WU, U9 TS5A3357DCUR

Commit message: Projector PCB!
Other:
- note added: "This is a separate PCB"
- note removed: "Delete this copy!"
Changed lines of the file:
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@@
 		)
 	)
-	(text "Delete this copy!"
+	(text "This is a separate PCB"
 		(exclude_from_sim no)
 		(at 54.102 21.59 0)
