File: KiCad/ImpulsWerk-Controller/ImpulsWerk-Controller.kicad_pcb (KiCad board)
At the start: 2 copper layers, 56.4 x 94.2 mm, 95 parts, among them CN2 PJ-307N5, J2 to DIN-6 Male, J3 Pause Button, J4 ICSP, J5 LED-Connector, Q1 AO3400A, Q2 SS8050, Q3 SS8050, Q4 SS8050, SW1 Guide/Follow, SW2 Mode -, SW3 Mode +, SW4 Frame -, SW5 Frame +, U1 ECS-TXO-3225MV-160-TR, U2 AP2210N-3.3TRG1, U3 74HCT14, U4 G3VM-61VY3(TR), U5 MCP4725, U6 LMC6482, U7 ATmega328P-A

Commit message: Before renaming
Parts:
- D8: footprint Peacemans Teile:OLED_128x63_i2c_0.96 -> easyEDA:HDR-TH_4P-P2.54-V-F
- SW2, SW3, SW4, SW5: footprint easyEDA:KEY-SMD_4P-L6.0-W6.0-P4.50-LS8.6 -> easyEDA:SW-SMD_4P-L6.0-W6.0-P4.50-LS9.0-H11.5
- moved D8 11.5 mm to (66.5, 46.4)
Other:
- board text added: "Clockwork Controller"
- board text added: "Crystal Clock & ESS Precision for Vintage Projectors by filmkorn.org"
- board text added: "Rev.A"
- board text removed: "Crystal Clock & ESS Precision for Vintage Projectors"
- board text removed: "Impulswerk Controller"
- board text removed: "Rev.A by filmkorn.org"
