File: KiCad/ImpulsWerk-Controller/ImpulsWerk-Controller.kicad_sch (KiCad schematic)
At the start: 96 parts, among them CN2 PJ-307N5, J1 DIN-6 male, J2 to DIN-6 Male, J3 Pause Button, J4 ICSP, J5 LED-Connector, Q1 AO3400A, Q2 SS8050, Q3 SS8050, Q4 SS8050, SW1 Guide/Follow, SW2 Mode -, SW3 Mode +, SW4 Frame -, SW5 Frame +, U1 ECS-TXO-3225MV-160-TR, U2 AP2210N-3.3TRG1, U3 74HCT14, U4 G3VM-61VY3(TR), U5 MCP4725, U6 LMC6482, U7 ATmega328P-A

Commit message: Before renaming
Parts:
- D8: footprint Peacemans Teile:OLED_128x63_i2c_0.96 -> easyEDA:HDR-TH_4P-P2.54-V-F; LCSC (none) -> C42163122
- SW2, SW3, SW4, SW5: footprint easyEDA:KEY-SMD_4P-L6.0-W6.0-P4.50-LS8.6 -> easyEDA:SW-SMD_4P-L6.0-W6.0-P4.50-LS9.0-H11.5; LCSC C455116 -> C455123
Other:
- title: SynCrystal Controller -> ImpulsWerk Controller
Changed lines of the file:
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@@
 	(paper "A3")
 	(title_block
-		(title "SynCrystal Controller")
+		(title "ImpulsWerk Controller")
 		(date "2025-02-11")
 		(rev "Rev.A")
@@
 			)
 		)
-		(property "Footprint" "easyEDA:KEY-SMD_4P-L6.0-W6.0-P4.50-LS8.6"
+		(property "Footprint" "easyEDA:SW-SMD_4P-L6.0-W6.0-P4.50-LS9.0-H11.5"
 			(at 231.14 250.19 0)
 			(effects
@@
 			)
 		)
-		(property "LCSC" "C455116"
+		(property "LCSC" "C455123"
 			(at 231.14 240.03 0)
 			(effects
@@
 			)
 		)
-		(property "Footprint" "easyEDA:KEY-SMD_4P-L6.0-W6.0-P4.50-LS8.6"
+		(property "Footprint" "easyEDA:SW-SMD_4P-L6.0-W6.0-P4.50-LS9.0-H11.5"
 			(at 231.14 267.97 0)
 			(effects
@@
 			)
 		)
-		(property "LCSC" "C455116"
+		(property "LCSC" "C455123"
 			(at 231.14 257.81 0)
 			(effects
@@
 			)
 		)
-		(property "Footprint" "easyEDA:KEY-SMD_4P-L6.0-W6.0-P4.50-LS8.6"
+		(property "Footprint" "easyEDA:SW-SMD_4P-L6.0-W6.0-P4.50-LS9.0-H11.5"
 			(at 231.14 276.86 0)
 			(effects
@@
 			)
 		)
-		(property "LCSC" "C455116"
+		(property "LCSC" "C455123"
 			(at 231.14 266.7 0)
 			(effects
@@
 			)
 		)
-		(property "Footprint" "Peacemans Teile:OLED_128x63_i2c_0.96"
+		(property "Footprint" "easyEDA:HDR-TH_4P-P2.54-V-F"
 			(at 193.04 247.65 90)
 			(effects
@@
 			)
 		)
-		(property "Datasheet" ""
+		(property "Datasheet" "https://www.lcsc.com/datasheet/lcsc_datasheet_2501071555_Hong-Cheng-HC-PM254-5-0H-1x4PZ-02A_C42163122.pdf"
 			(at 193.04 247.65 90)
 			(effects
@@
 			)
 		)
+		(property "LCSC" "C42163122"
+			(at 186.69 254 0)
+			(effects
+				(font
+					(size 1.27 1.27)
+				)
+				(hide yes)
+			)
+		)
 		(pin "1"
 		)
@@
 			)
 		)
-		(property "Footprint" "easyEDA:KEY-SMD_4P-L6.0-W6.0-P4.50-LS8.6"
+		(property "Footprint" "easyEDA:SW-SMD_4P-L6.0-W6.0-P4.50-LS9.0-H11.5"
 			(at 231.14 259.08 0)
 			(effects
@@
 			)
 		)
-		(property "LCSC" "C455116"
+		(property "LCSC" "C455123"
 			(at 231.14 248.92 0)
 			(effects
