File: KiCad/ImpulsWerk-Frontpanel/ImpulsWerk-Frontpanel.kicad_sch (KiCad schematic)
At the start: 7 parts

Commit message: Before renaming
Parts:
- added H1, H2, H3, H4, H5, H6, H7, H8: MountingHole, MountingHole:MountingHole_3.2mm_M3_DIN965, symbol Mechanical:MountingHole
- D1: value no sync -> no sync (re); footprint LED_SMD:LED_0805_2012Metric -> easyEDA:LED-SMD_L3.2-W1.6-FD_EH-GREEN-1; LCSC C2297 -> C2892757
- D2: value Crystal -> Crystal (gr); footprint LED_SMD:LED_0805_2012Metric -> easyEDA:LED-SMD_L3.2-W1.6-FD_EH-GREEN-1; LCSC C2297 -> C2980185
- D3: value Ext. Imp. -> Ext. Imp. (or); footprint LED_SMD:LED_0805_2012Metric -> (none); LCSC C2297 -> C424133
- J1: footprint easyEDA:HDR-SMD_HX-PM2.54-1X4P-TP-YQ -> easyEDA:HDR-SMD_6P-P2.00-V-M-R2-C3-LS6.5; symbol Connector:Conn_01x04_Pin -> easyEDA:PZ200-2-03-S; LCSC (none) -> C3294482; LCSC Part (none) -> C3294482
- R1, R2: LCSC C26010 -> C22978
- R3: LCSC C26010 -> C21190
Connections:
- net GND: now also J1.2, J1.6
- net at R2.1: now also J1.3; no longer J1.2 (Pin_2)
- net at R3.2: now also J1.5; no longer J1.3 (Pin_3)
